File: cursed-scandinavian-iso-van.kicad_pcb (KiCad board)
At the start: 2 copper layers, 105 parts, among them J1 Conn_01x04, SW1 SW_Push, U1 ATmega32U4-A, Y1 16MHz

Commit message: rerouted everything again
Parts:
- moved SW1 58.7 mm to (111.1, 76.4), turned to 180 degrees
- moved R1 46.0 mm to (117.5, 78.6), turned to 45 degrees
- moved C7 21.8 mm to (118.3, 93.7), turned to -90 degrees
- moved C6 21.4 mm to (131.8, 96.0), turned to 180 degrees
- moved R4 20.0 mm to (135.7, 92.8)
- moved Y1 19.4 mm to (127.0, 76.8), turned to 180 degrees
- moved C1 18.6 mm to (117.6, 88.1), turned to 180 degrees
- moved C3 18.3 mm to (123.0, 76.8), turned to 90 degrees
- moved C2 17.5 mm to (131.0, 76.8), turned to -90 degrees
- moved C4 7.03 mm to (135.7, 84.1), turned to 135 degrees
- moved R3 6.40 mm to (213.5, 44.5)
- moved C5 6.35 mm to (119.1, 81.6), turned to 90 degrees
- moved R2 6.05 mm to (213.5, 41.3)
- moved U1 3.61 mm to (127.0, 88.0), turned to 0 degrees
- moved F1 3.40 mm to (214.9, 46.8)
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Routing:
- net Net-(U1-D-): track 0.00 -> 223.4 mm, vias 0 -> 2
- net Net-(U1-D+): track 0.00 -> 217.9 mm, vias 0 -> 2
- net GND: track 0.00 -> 77.3 mm
- net +5V: track 0.00 -> 69.4 mm, vias 0 -> 5
- net Net-(U1-~{RESET}): track 0.00 -> 16.6 mm, vias 0 -> 2
- net XTAL2: track 0.00 -> 10.3 mm
- net XTAL1: track 0.00 -> 8.57 mm
- net VCC: track 0.00 -> 5.19 mm
- net Net-(D11-A): track 4.49 -> 0.00 mm
- net Net-(D23-A): track 4.49 -> 0.00 mm
- net Net-(D21-A): track 4.49 -> 0.00 mm
- net Net-(D22-A): track 4.49 -> 0.00 mm
- net Net-(D9-A): track 4.49 -> 0.00 mm
- net Net-(D10-A): track 4.49 -> 0.00 mm
- net D+: track 0.00 -> 4.34 mm
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Other:
- board outline added: 241.3 x 74.6 mm

Commit message: maybe all the columns
Connections:
- SW1 pad 1: GND -> Net-(U1-~{RESET})
- SW1 pad 2: Net-(U1-~{RESET}) -> GND
- U1 pad 10: unconnected-(U1-PB2-Pad10) -> COL2
- U1 pad 11: unconnected-(U1-PB3-Pad11) -> COL3
- U1 pad 18: unconnected-(U1-PD0-Pad18) -> COL4
- U1 pad 19: unconnected-(U1-PD1-Pad19) -> COL5
- U1 pad 20: unconnected-(U1-PD2-Pad20) -> COL6
- U1 pad 21: unconnected-(U1-PD3-Pad21) -> COL7
- U1 pad 22: unconnected-(U1-PD5-Pad22) -> COL8
- U1 pad 29: unconnected-(U1-PB5-Pad29) -> COL9
- U1 pad 30: unconnected-(U1-PB6-Pad30) -> COL10
- U1 pad 31: unconnected-(U1-PC6-Pad31) -> COL11
- U1 pad 32: unconnected-(U1-PC7-Pad32) -> ROW3
- U1 pad 8: unconnected-(U1-PB0-Pad8) -> COL0
- U1 pad 9: unconnected-(U1-PB1-Pad9) -> COL1
Routing:
- net ROW3: track 0.00 -> 236.3 mm
- net ROW1: track 0.00 -> 229.4 mm
- net ROW0: track 0.00 -> 223.8 mm
- net ROW2: track 0.00 -> 221.7 mm
- net COL11: track 0.00 -> 183.3 mm, vias 0 -> 1
- net COL10: track 0.00 -> 169.8 mm, vias 0 -> 1
- net COL0: track 0.00 -> 153.4 mm, vias 0 -> 1
- net COL9: track 0.00 -> 147.3 mm, vias 0 -> 1
- net COL1: track 0.00 -> 141.0 mm, vias 0 -> 1
- net COL8: track 0.00 -> 130.9 mm, vias 0 -> 1
- net COL2: track 0.00 -> 99.3 mm, vias 0 -> 1
- net COL7: track 0.00 -> 94.7 mm, vias 0 -> 1
- net COL3: track 0.00 -> 90.8 mm, vias 0 -> 1
- net COL6: track 0.00 -> 87.0 mm, vias 0 -> 1
- net COL4: track 0.00 -> 73.2 mm, vias 0 -> 1
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
Commit message: only silk and edge complaints
Parts:
- moved C6 1.12 mm to (131.0, 96.8)
Connections:
- U1 pad 26: unconnected-(U1-PD6-Pad26) -> ROW0
- U1 pad 27: unconnected-(U1-PD7-Pad27) -> ROW1
- U1 pad 28: unconnected-(U1-PB4-Pad28) -> ROW2
Routing:
- net +5V: track 71.6 -> 257.2 mm, vias 5 -> 7
- net ROW1: track 229.4 -> 326.4 mm, vias 0 -> 2
- net ROW2: track 221.7 -> 304.8 mm
- net ROW0: track 223.8 -> 305.0 mm, vias 0 -> 2
- net GND: track 77.3 -> 101.0 mm, vias 0 -> 1
- net unconnected-(U1-PB4-Pad28): track 18.8 -> 0.00 mm
- net unconnected-(U1-PD7-Pad27): track 17.7 -> 0.00 mm
- net unconnected-(U1-PD6-Pad26): track 17.7 -> 0.00 mm
- net Net-(U1-~{RESET}): track 16.6 -> 23.0 mm, vias 2 -> 3
- net Net-(U1-D-): track 222.6 -> 224.6 mm
- net Net-(U1-D+): track 217.0 -> 218.7 mm
- net COL9: track 147.3 -> 145.9 mm
- net XTAL1: track 8.57 -> 7.81 mm
- added copper zone on B.Cu, net GND
- added copper zone on F.Cu, net GND
