File: cursed-scandinavian-iso-van.kicad_pcb (KiCad board)
At the start: 2 copper layers, 241.3 x 74.6 mm, 105 parts, among them J1 Conn_01x04, SW1 SW_Push, U1 ATmega32U4-A, Y1 16MHz

Commit message: second attempt
Parts:
- C1, C2, C3, C4, C5, C6, C7: footprint Capacitor_SMD:C_0805_2012Metric -> Capacitor_SMD:C_0402_1005Metric
- R1, R2, R3, R4: footprint Resistor_SMD:R_0805_2012Metric -> Resistor_SMD:R_0402_1005Metric
- S3: value MX_stab -> locked
- U1: value ATmega32U4-A -> ATmega32U4-M; footprint Package_QFP:TQFP-44_10x10mm_P0.8mm -> Package_DFN_QFN:QFN-44-1EP_7x7mm_P0.5mm_EP5.2x5.2mm
- moved SW1 135.8 mm to (246.9, 78.9), turned to 0 degrees
- moved C7 95.4 mm to (211.9, 75.4), turned to 90 degrees
- moved R1 93.8 mm to (211.1, 83.1), turned to -90 degrees
- moved C1 93.0 mm to (210.3, 81.0), turned to 90 degrees
- moved C5 86.0 mm to (204.8, 74.6), turned to 180 degrees
- moved C3 85.5 mm to (207.6, 89.5), turned to -90 degrees
- moved C6 79.8 mm to (209.6, 83.1), turned to 90 degrees
- moved Y1 78.7 mm to (204.7, 89.5), turned to 0 degrees
- moved U1 76.0 mm to (202.6, 79.8), turned to 180 degrees
- moved C2 72.1 mm to (202.0, 89.5), turned to 90 degrees
- moved R4 64.1 mm to (197.6, 76.2), turned to 90 degrees
- moved C4 61.6 mm to (197.3, 83.0), turned to -45 degrees
- moved R2 38.2 mm to (210.9, 79.4), turned to 180 degrees
- moved R3 33.6 mm to (210.9, 77.9), turned to 180 degrees
- moved F1 1.12 mm to (215.7, 46.0)
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- renumbered MX33 to locked
Connections:
- U1 pad 10: COL2 -> unconnected-(U1-PB2-Pad10)
- U1 pad 11: COL3 -> unconnected-(U1-PB3-Pad11)
- U1 pad 18: COL4 -> COL9
- U1 pad 19: COL5 -> COL10
- U1 pad 20: COL6 -> COL11
- U1 pad 21: COL7 -> COL8
- U1 pad 22: COL8 -> ROW3
- U1 pad 25: unconnected-(U1-PD4-Pad25) -> COL0
- U1 pad 26: ROW0 -> COL1
- U1 pad 27: ROW1 -> COL2
- U1 pad 28: ROW2 -> COL3
- U1 pad 29: COL9 -> COL4
- U1 pad 30: COL10 -> COL5
- U1 pad 31: COL11 -> COL6
- U1 pad 32: ROW3 -> COL7
- U1 pad 36: unconnected-(U1-PF7-Pad36) -> ROW2
- U1 pad 37: unconnected-(U1-PF6-Pad37) -> ROW1
- U1 pad 38: unconnected-(U1-PF5-Pad38) -> ROW0
- U1 pad 8: COL0 -> unconnected-(U1-PB0-Pad8)
- U1 pad 9: COL1 -> unconnected-(U1-PB1-Pad9)
Routing:
- net Net-(U1-D-): track 224.6 -> 4.60 mm, vias 4 -> 0
- net Net-(U1-D+): track 218.7 -> 4.70 mm, vias 4 -> 0
- net +5V: track 257.2 -> 115.9 mm
- net ROW2: track 304.8 -> 225.4 mm, vias 0 -> 4
- net COL3: track 90.8 -> 166.9 mm
- net COL0: track 153.4 -> 229.3 mm
- net COL2: track 99.3 -> 173.2 mm
- net COL1: track 141.0 -> 213.0 mm
- net ROW1: track 326.4 -> 255.0 mm, vias 2 -> 4
- net D+: track 3.93 -> 70.5 mm
- net D-: track 3.93 -> 68.8 mm
- net COL4: track 73.2 -> 134.3 mm
- net COL9: track 145.9 -> 85.2 mm, vias 1 -> 0
- net COL10: track 169.7 -> 110.3 mm
- net COL5: track 59.2 -> 114.7 mm
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Other:
- board text removed: "Moonchild Keyboards - Cursed Scandinavian ISO Van"

Commit message: tuned data line
Routing:
- net D-: track 68.8 -> 70.5 mm
- net +5V: track 115.9 -> 114.5 mm

Commit message: maybe
Parts:
- removed F1: 500mA, Fuse:Fuse_1206_3216Metric
- removed R2, R3: 22, Resistor_SMD:R_0402_1005Metric
- removed R4: 10k, Resistor_SMD:R_0402_1005Metric
- removed Y1: 16MHz, Crystal:Crystal_SMD_3225-4Pin_3.2x2.5mm
- added C8: 1uF, Capacitor_SMD:C_0402_1005Metric, B.Cu at (213.2, 45.2)
- added C9: 1uF, Capacitor_SMD:C_0402_1005Metric, B.Cu at (213.4, 50.8)
- added U2: XC6206PxxxMR, Package_TO_SOT_SMD:SOT-23-3, B.Cu at (213.2, 48.1)
- C1: value 1u -> 100nF
- C2, C3: value 22p -> 100nF
- C4, C5, C6: value 0.1u -> 100nF
- C7: value 10u -> 10uF; footprint Capacitor_SMD:C_0402_1005Metric -> Capacitor_SMD:C_0603_1608Metric
- SW1: footprint Button_Switch_SMD:SW_SPST_TL3342 -> Button_Switch_SMD:SW_SPST_SKQG_WithoutStem
- U1: value ATmega32U4-M -> STM32F072CBTx; footprint Package_DFN_QFN:QFN-44-1EP_7x7mm_P0.5mm_EP5.2x5.2mm -> Package_QFP:LQFP-48_7x7mm_P0.5mm
- moved C2 59.0 mm to (222.2, 34.1), turned to -135 degrees
- moved C4 55.8 mm to (230.4, 38.1), turned to 135 degrees
- moved R1 54.1 mm to (241.3, 38.1)
- moved C6 47.8 mm to (230.8, 40.3), turned to 45 degrees
- moved C3 47.4 mm to (218.2, 43.2), turned to -45 degrees
- moved U1 45.0 mm to (224.4, 40.5), turned to 135 degrees
- moved C1 39.5 mm to (229.7, 46.5), turned to -135 degrees
- moved SW1 39.2 mm to (247.4, 39.8)
- moved C5 37.2 mm to (228.6, 46.0), turned to 45 degrees
- moved C7 32.1 mm to (216.7, 43.7), turned to -45 degrees
Connections:
- C1 pad 1: Net-(U1-UCAP) -> NRST
- C2 pad 1: GND -> +3.3V
- C2 pad 2: XTAL1 -> GND
- C3 pad 1: GND -> +3.3V
- C3 pad 2: XTAL2 -> GND
- C4 pad 1: +5V -> +3.3V
- C5 pad 1: +5V -> +3.3V
- C6 pad 1: +5V -> +3.3V
- C7 pad 1: +5V -> +3.3V
- J1 pad 1: VCC -> +5V
- J1 pad 2: D- -> D_N
- J1 pad 3: D+ -> D_P
- R1 pad 1: +5V -> BOOT0
- R1 pad 2: Net-(U1-~{RESET}) -> GND
- SW1 pad 1: Net-(U1-~{RESET}) -> +3.3V
- SW1 pad 2: GND -> BOOT0
- U1 pad 1: unconnected-(U1-PE6-Pad1) -> +3.3V
- U1 pad 10: unconnected-(U1-PB2-Pad10) -> ROW3
- U1 pad 11: unconnected-(U1-PB3-Pad11) -> ROW2
- U1 pad 12: unconnected-(U1-PB7-Pad12) -> ROW1
- U1 pad 13: Net-(U1-~{RESET}) -> COL0
- U1 pad 14: +5V -> COL1
- U1 pad 15: GND -> COL2
- U1 pad 16: XTAL2 -> COL3
- U1 pad 17: XTAL1 -> COL4
- U1 pad 18: COL9 -> COL5
- U1 pad 19: COL10 -> COL6
- U1 pad 2: +5V -> unconnected-(U1-PC13-Pad2)
- U1 pad 20: COL11 -> COL7
- U1 pad 22: ROW3 -> unconnected-(U1-PB11-Pad22)
- U1 pad 24: +5V -> +3.3V
- U1 pad 25: COL0 -> COL9
- U1 pad 26: COL1 -> ROW0
- U1 pad 27: COL2 -> unconnected-(U1-PB14-Pad27)
- U1 pad 28: COL3 -> unconnected-(U1-PB15-Pad28)
- U1 pad 29: COL4 -> unconnected-(U1-PA8-Pad29)
- U1 pad 3: Net-(U1-D-) -> COL11
- U1 pad 30: COL5 -> unconnected-(U1-PA9-Pad30)
- U1 pad 31: COL6 -> unconnected-(U1-PA10-Pad31)
- U1 pad 32: COL7 -> D_N
- U1 pad 33: Net-(U1-~{HWB}/PE2) -> D_P
- U1 pad 34: +5V -> unconnected-(U1-PA13-Pad34)
- U1 pad 36: ROW2 -> +3.3V
- U1 pad 37: ROW1 -> unconnected-(U1-PA14-Pad37)
- U1 pad 38: ROW0 -> unconnected-(U1-PA15-Pad38)
- U1 pad 4: Net-(U1-D+) -> COL10
- U1 pad 43: GND -> unconnected-(U1-PB7-Pad43)
- U1 pad 44: +5V -> BOOT0
- U1 pad 45: GND -> unconnected-(U1-PB8-Pad45)
- U1 pad 5: GND -> unconnected-(U1-PF0-Pad5)
- U1 pad 6: Net-(U1-UCAP) -> unconnected-(U1-PF1-Pad6)
- U1 pad 7: +5V -> NRST
- U1 pad 8: unconnected-(U1-PB0-Pad8) -> GND
- U1 pad 9: unconnected-(U1-PB1-Pad9) -> +3.3V
Routing:
- net +5V: track 114.5 -> 6.52 mm, vias 7 -> 0
- net +3.3V: track 0.00 -> 87.8 mm, vias 0 -> 7
- net D-: track 70.5 -> 0.00 mm
- net D+: track 70.5 -> 0.00 mm
- net Net-(U1-~{RESET}): track 48.2 -> 0.00 mm
- net COL11: track 131.4 -> 85.1 mm, vias 1 -> 0
- net COL10: track 110.3 -> 67.0 mm, vias 1 -> 0
- net ROW0: track 271.5 -> 233.0 mm
- net COL3: track 166.9 -> 204.4 mm
- net ROW3: track 238.0 -> 274.1 mm
- net GND: track 95.1 -> 59.2 mm
- net COL0: track 229.3 -> 262.8 mm
- net COL1: track 213.0 -> 244.1 mm
- net COL7: track 75.4 -> 105.6 mm
- net COL4: track 134.3 -> 164.3 mm
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