File: cursed-scandinavian-iso-van.kicad_pcb (KiCad board)
At the start: 2 copper layers, 241.3 x 74.6 mm, 105 parts, among them J1 Conn_01x04, SW1 SW_Push, U1 ATmega32U4-M, Y1 16MHz

Commit message: finish PCB in STM32
Parts:
- removed J1: Conn_01x04, Connector_JST:JST_SH_SM04B-SRSS-TB_1x04-1MP_P1.00mm_Horizontal
- removed R2, R3: 22, Resistor_SMD:R_0402_1005Metric
- removed R4: 10k, Resistor_SMD:R_0402_1005Metric
- removed Y1: 16MHz, Crystal:Crystal_SMD_3225-4Pin_3.2x2.5mm
- added C10: 100nF, Capacitor_SMD:C_0402_1005Metric, B.Cu at (218.6, 43.7)
- added C8: 1uF, Capacitor_SMD:C_0402_1005Metric, B.Cu at (221.5, 40.1)
- added C9: 1uF, Capacitor_SMD:C_0402_1005Metric, B.Cu at (221.5, 42.0)
- added J2: Conn_01x04_Socket, Connector_JST:JST_SH_SM04B-SRSS-TB_1x04-1MP_P1.00mm_Horizontal, B.Cu at (209.9, 41.3)
- added U2: PRTR5V0U2X, Package_TO_SOT_SMD:SOT-143, B.Cu at (215.4, 40.9)
- added U3: XC6206P332MR-Regulator_Linear, Package_TO_SOT_SMD:SOT-23, B.Cu at (219.1, 40.9)
- C1: value 1u -> 100nF
- C2, C3: value 22p -> 100nF
- C4, C5: value 0.1u -> 100nF
- C6: value 0.1u -> 10uF; footprint Capacitor_SMD:C_0402_1005Metric -> Capacitor_SMD:C_0603_1608Metric
- C7: value 10u -> 100nF
- F1: value 500mA -> ASMD1206-150
- SW1: value SW_Push -> SKQGABE010; footprint Button_Switch_SMD:SW_SPST_TL3342 -> Button_Switch_SMD:SW_SPST_SKQG_WithoutStem
- U1: value ATmega32U4-M -> STM32F072CBU6; footprint Package_DFN_QFN:QFN-44-1EP_7x7mm_P0.5mm_EP5.2x5.2mm -> Package_QFP:LQFP-48-1EP_7x7mm_P0.5mm_EP3.6x3.6mm
- moved R1 24.7 mm to (235.6, 79.0), turned to 90 degrees
- moved C7 14.9 mm to (204.2, 88.2), turned to 0 degrees
- moved C5 7.24 mm to (198.9, 78.8)
- moved C2 7.16 mm to (208.3, 86.2), turned to 0 degrees
- moved C4 6.65 mm to (201.5, 88.2), turned to 180 degrees
- moved SW1 6.56 mm to (240.3, 79.0), turned to 180 degrees
- moved C6 5.38 mm to (208.4, 77.8)
- moved C1 4.42 mm to (207.2, 77.8)
- moved U1 2.92 mm to (203.6, 82.5), turned to 90 degrees
- moved F1 2.27 mm to (215.7, 43.8)
- moved C3 1.89 mm to (207.2, 87.6)
Connections:
- C1 pad 1: Net-(U1-UCAP) -> +3V3
- C2 pad 1: GND -> +3V3
- C2 pad 2: XTAL1 -> GND
- C3 pad 1: GND -> +3V3
- C3 pad 2: XTAL2 -> GND
- C4 pad 1: +5V -> +3V3
- C5 pad 1: +5V -> +3V3
- C6 pad 1: +5V -> +3V3
- C7 pad 1: +5V -> NRST
- D1 pad 1: ROW0 -> row0
- D10 pad 1: ROW0 -> row0
- D11 pad 1: ROW0 -> row0
- D12 pad 1: ROW0 -> row0
- D13 pad 1: ROW1 -> row1
- D14 pad 1: ROW1 -> row1
- D15 pad 1: ROW1 -> row1
- D16 pad 1: ROW1 -> row1
- D17 pad 1: ROW1 -> row1
- D18 pad 1: ROW1 -> row1
- D19 pad 1: ROW1 -> row1
- D2 pad 1: ROW0 -> row0
- D20 pad 1: ROW1 -> row1
- D21 pad 1: ROW1 -> row1
- D22 pad 1: ROW1 -> row1
- D23 pad 1: ROW1 -> row1
- D24 pad 1: ROW1 -> row1
- D25 pad 1: ROW2 -> row2
- D26 pad 1: ROW2 -> row2
- D27 pad 1: ROW2 -> row2
- D28 pad 1: ROW2 -> row2
- D29 pad 1: ROW2 -> row2
- D3 pad 1: ROW0 -> row0
- D30 pad 1: ROW2 -> row2
- D31 pad 1: ROW2 -> row2
- D32 pad 1: ROW2 -> row2
- D33 pad 1: ROW2 -> row2
- D34 pad 1: ROW2 -> row2
- D35 pad 1: ROW2 -> row2
- D36 pad 1: ROW3 -> row3
- D37 pad 1: ROW3 -> row3
- D38 pad 1: ROW3 -> row3
- D39 pad 1: ROW3 -> row3
- D4 pad 1: ROW0 -> row0
- D40 pad 1: ROW3 -> row3
- D41 pad 1: ROW3 -> row3
- D42 pad 1: ROW3 -> row3
- D43 pad 1: ROW3 -> row3
- D5 pad 1: ROW0 -> row0
- D6 pad 1: ROW0 -> row0
- D7 pad 1: ROW0 -> row0
- D8 pad 1: ROW0 -> row0
- D9 pad 1: ROW0 -> row0
- F1 pad 1: VCC -> VBUS
- MX1 pad 1: COL0 -> col0
- MX10 pad 1: COL9 -> col9
- MX11 pad 1: COL10 -> col10
- MX12 pad 1: COL11 -> col11
- MX13 pad 1: COL0 -> col0
- MX14 pad 1: COL1 -> col1
- MX15 pad 1: COL2 -> col2
- MX16 pad 1: COL3 -> col3
- MX17 pad 1: COL4 -> col4
- MX18 pad 1: COL5 -> col5
- MX19 pad 1: COL6 -> col6
- MX2 pad 1: COL1 -> col1
- MX20 pad 1: COL7 -> col7
- MX21 pad 1: COL8 -> col8
- MX22 pad 1: COL9 -> col9
- MX23 pad 1: COL10 -> col10
- MX24 pad 1: COL11 -> col11
- MX25 pad 1: COL0 -> col0
- MX26 pad 1: COL1 -> col1
- MX27 pad 1: COL2 -> col2
- MX28 pad 1: COL3 -> col3
- MX29 pad 1: COL4 -> col4
- MX3 pad 1: COL2 -> col2
- MX30 pad 1: COL5 -> col5
- MX31 pad 1: COL6 -> col6
- MX32 pad 1: COL7 -> col7
- MX34 pad 1: COL10 -> col10
- MX35 pad 1: COL11 -> col11
- MX36 pad 1: COL0 -> col0
- MX37 pad 1: COL1 -> col1
- MX38 pad 1: COL3 -> col3
- MX39 pad 1: COL6 -> col6
- MX4 pad 1: COL3 -> col3
- MX40 pad 1: COL8 -> col8
- MX41 pad 1: COL9 -> col9
- MX42 pad 1: COL10 -> col10
- MX43 pad 1: COL11 -> col11
- MX5 pad 1: COL4 -> col4
- MX6 pad 1: COL5 -> col5
- MX7 pad 1: COL6 -> col6
- MX8 pad 1: COL7 -> col7
- MX9 pad 1: COL8 -> col8
- R1 pad 1: +5V -> BOOT0
- R1 pad 2: Net-(U1-~{RESET}) -> GND
- SW1 pad 1: Net-(U1-~{RESET}) -> +3V3
- SW1 pad 2: GND -> BOOT0
- U1 pad 1: unconnected-(U1-PE6-Pad1) -> +3V3
- U1 pad 10: unconnected-(U1-PB2-Pad10) -> /A0
- U1 pad 11: unconnected-(U1-PB3-Pad11) -> /A1
- U1 pad 12: unconnected-(U1-PB7-Pad12) -> /A2
- U1 pad 13: Net-(U1-~{RESET}) -> row3
- U1 pad 14: +5V -> col8
- U1 pad 15: GND -> col7
- U1 pad 16: XTAL2 -> col6
- U1 pad 17: XTAL1 -> col5
- U1 pad 18: COL9 -> col4
- U1 pad 19: COL10 -> col3
- U1 pad 2: +5V -> unconnected-(U1-PC13-Pad2)
- U1 pad 20: COL11 -> col2
- U1 pad 21: COL8 -> col1
- U1 pad 22: ROW3 -> col0
- U1 pad 24: +5V -> +3V3
- U1 pad 25: COL0 -> row2
- U1 pad 26: COL1 -> row0
- U1 pad 27: COL2 -> /B14
- U1 pad 28: COL3 -> /B15
- U1 pad 29: COL4 -> /A8
- U1 pad 3: Net-(U1-D-) -> unconnected-(U1-PC14-Pad3)
- U1 pad 30: COL5 -> /A9
- U1 pad 31: COL6 -> /A10
- U1 pad 32: COL7 -> D_N
- U1 pad 33: Net-(U1-~{HWB}/PE2) -> D_P
- U1 pad 34: +5V -> row1
- U1 pad 36: ROW2 -> +3V3
- U1 pad 37: ROW1 -> /A14
- U1 pad 38: ROW0 -> /A15
- U1 pad 39: unconnected-(U1-PF4-Pad39) -> /B3
- U1 pad 4: Net-(U1-D+) -> unconnected-(U1-PC15-Pad4)
- U1 pad 40: unconnected-(U1-PF1-Pad40) -> /B4
- U1 pad 41: unconnected-(U1-PF0-Pad41) -> /B5
- U1 pad 42: unconnected-(U1-AREF-Pad42) -> /B6
- U1 pad 43: GND -> /B7
- U1 pad 44: +5V -> BOOT0
- U1 pad 45: GND -> /B8
- U1 pad 5: GND -> unconnected-(U1-PF0-Pad5)
- U1 pad 6: Net-(U1-UCAP) -> unconnected-(U1-PF1-Pad6)
- U1 pad 7: +5V -> NRST
- U1 pad 8: unconnected-(U1-PB0-Pad8) -> GND
- U1 pad 9: unconnected-(U1-PB1-Pad9) -> +3V3
- locked pad 1: COL8 -> col8
Routing:
- net ROW0: track 271.5 -> 0.00 mm
- net row0: track 0.00 -> 267.0 mm, vias 0 -> 1
- net ROW1: track 255.0 -> 0.00 mm, vias 4 -> 0
- net row1: track 0.00 -> 242.5 mm, vias 0 -> 2
- net col0: track 0.00 -> 238.6 mm
- net ROW3: track 238.0 -> 0.00 mm, vias 2 -> 0
- net row3: track 0.00 -> 235.7 mm, vias 0 -> 1
- net COL0: track 229.3 -> 0.00 mm, vias 1 -> 0
- net row2: track 0.00 -> 227.9 mm, vias 0 -> 2
- net ROW2: track 225.4 -> 0.00 mm, vias 4 -> 0
- net col1: track 0.00 -> 218.9 mm
- net COL1: track 213.0 -> 0.00 mm, vias 1 -> 0
- net col3: track 0.00 -> 174.9 mm
- net col2: track 0.00 -> 173.3 mm, vias 0 -> 1
- net COL2: track 173.2 -> 0.00 mm, vias 1 -> 0
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Other:
- board text added: "RESET"
- board text added: "ScandiVan"
- board text added: "by Ciantha and jlw"
- board text added: "v1 [2024-01]"

Commit message: updated PCB
Connections:
- U1 pad 43: /B7 -> col10
- U1 pad 45: /B8 -> col11
- U1 pad 46: /B9 -> col9
Routing:
- net col11: track 58.1 -> 107.3 mm
- net col10: track 58.1 -> 94.1 mm, vias 0 -> 1
- net GND: track 22.5 -> 37.1 mm, vias 23 -> 29
- net col9: track 57.6 -> 66.7 mm
Changed lines of the file:
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@@
   (net 82 "/B4")
   (net 83 "/B5")
-  (net 84 "/B7")
-  (net 85 "/B8")
-  (net 86 "/B9")
-  (net 87 "/A15")
-  (net 88 "/A14")
-  (net 89 "/B6")
+  (net 84 "/A15")
+  (net 85 "/A14")
+  (net 86 "/B6")
   (footprint "PCM_marbastlib-mx:STAB_MX_P_3u" (layer "F.Cu")
     (at 95.25 90.4875 180)
@@
       (net 46 "+3V3") (pinfunction "VDDIO2") (pintype "power_in"))
     (pad "37" smd roundrect (at 2.75 4.1625 90) (size 0.3 1.475) (layers "B.Cu" "B.Paste" "B.Mask") (roundrect_rratio 0.25)
-      (net 88 "/A14") (pinfunction "PA14") (pintype "bidirectional"))
+      (net 85 "/A14") (pinfunction "PA14") (pintype "bidirectional"))
     (pad "38" smd roundrect (at 2.25 4.1625 90) (size 0.3 1.475) (layers "B.Cu" "B.Paste" "B.Mask") (roundrect_rratio 0.25)
-      (net 87 "/A15") (pinfunction "PA15") (pintype "bidirectional"))
+      (net 84 "/A15") (pinfunction "PA15") (pintype "bidirectional"))
     (pad "39" smd roundrect (at 1.75 4.1625 90) (size 0.3 1.475) (layers "B.Cu" "B.Paste" "B.Mask") (roundrect_rratio 0.25)
       (net 81 "/B3") (pinfunction "PB3") (pintype "bidirectional"))
@@
       (net 83 "/B5") (pinfunction "PB5") (pintype "bidirectional"))
     (pad "42" smd roundrect (at 0.25 4.1625 90) (size 0.3 1.475) (layers "B.Cu" "B.Paste" "B.Mask") (roundrect_rratio 0.25)
-      (net 89 "/B6") (pinfunction "PB6") (pintype "bidirectional"))
+      (net 86 "/B6") (pinfunction "PB6") (pintype "bidirectional"))
     (pad "43" smd roundrect (at -0.25 4.1625 90) (size 0.3 1.475) (layers "B.Cu" "B.Paste" "B.Mask") (roundrect_rratio 0.25)
-      (net 84 "/B7") (pinfunction "PB7") (pintype "bidirectional"))
+      (net 65 "col10") (pinfunction "PB7") (pintype "bidirectional"))
     (pad "44" smd roundrect (at -0.75 4.1625 90) (size 0.3 1.475) (layers "B.Cu" "B.Paste" "B.Mask") (roundrect_rratio 0.25)
       (net 67 "BOOT0") (pinfunction "BOOT0") (pintype "input"))
     (pad "45" smd roundrect (at -1.25 4.1625 90) (size 0.3 1.475) (layers "B.Cu" "B.Paste" "B.Mask") (roundrect_rratio 0.25)
-      (net 85 "/B8") (pinfunction "PB8") (pintype "bidirectional"))
+      (net 66 "col11") (pinfunction "PB8") (pintype "bidirectional"))
     (pad "46" smd roundrect (at -1.75 4.1625 90) (size 0.3 1.475) (layers "B.Cu" "B.Paste" "B.Mask") (roundrect_rratio 0.25)
-      (net 86 "/B9") (pinfunction "PB9") (pintype "bidirectional"))
+      (net 64 "col9") (pinfunction "PB9") (pintype "bidirectional"))
     (pad "47" smd roundrect (at -2.25 4.1625 90) (size 0.3 1.475) (layers "B.Cu" "B.Paste" "B.Mask") (roundrect_rratio 0.25)
       (net 1 "GND") (pinfunction "VSS") (pintype "passive"))
@@
   )
   (via (at 208.5 41.75) (size 0.8) (drill 0.4) (layers "F.Cu" "B.Cu") (net 1))
+  (via (at 203.6 82.5) (size 0.8) (drill 0.4) (layers "F.Cu" "B.Cu") (net 1))
   (via (at 94.7 86.45) (size 0.8) (drill 0.4) (layers "F.Cu" "B.Cu") (free) (net 1))
   (via (at 198.1005 79.723488) (size 0.8) (drill 0.4) (layers "F.Cu" "B.Cu") (net 1))
   (via (at 207.6 76.5) (size 0.8) (drill 0.4) (layers "F.Cu" "B.Cu") (net 1))
+  (via (at 230.7 84.5) (size 0.8) (drill 0.4) (layers "F.Cu" "B.Cu") (free) (net 1))
   (via (at 114.25 87.9) (size 0.8) (drill 0.4) (layers "F.Cu" "B.Cu") (free) (net 1))
   (via (at 54.7 86.45) (size 0.8) (drill 0.4) (layers "F.Cu" "B.Cu") (free) (net 1))
@@
   (via (at 222.15 39.627) (size 0.8) (drill 0.4) (layers "F.Cu" "B.Cu") (net 1))
   (via (at 219.15 44.227) (size 0.8) (drill 0.4) (layers "F.Cu" "B.Cu") (net 1))
+  (via (at 237.33125 85.725) (size 0.8) (drill 0.4) (layers "F.Cu" "B.Cu") (free) (net 1))
+  (via (at 211.4 80.9) (size 0.8) (drill 0.4) (layers "F.Cu" "B.Cu") (free) (net 1))
   (via (at 200.5 69.35) (size 0.8) (drill 0.4) (layers "F.Cu" "B.Cu") (free) (net 1))
   (via (at 75.95 87.3) (size 0.8) (drill 0.4) (layers "F.Cu" "B.Cu") (free) (net 1))
   (via (at 88.7 97.95) (size 0.8) (drill 0.4) (layers "F.Cu" "B.Cu") (free) (net 1))
+  (via (at 218.28125 85.725) (size 0.8) (drill 0.4) (layers "F.Cu" "B.Cu") (free) (net 1))
+  (via (at 230.7 78.9) (size 0.8) (drill 0.4) (layers "F.Cu" "B.Cu") (free) (net 1))
   (via (at 222.15 42.527) (size 0.8) (drill 0.4) (layers "F.Cu" "B.Cu") (net 1))
   (via (at 206.7 76.6) (size 0.8) (drill 0.4) (layers "F.Cu" "B.Cu") (net 1))
   (via (at 205.5 88.15) (size 0.8) (drill 0.4) (layers "F.Cu" "B.Cu") (net 1))
   (segment (start 205.85 78.3375) (end 205.85 79.176042) (width 0.3) (layer "B.Cu") (net 1))
+  (segment (start 201.35 80.25) (end 203.6 82.5) (width 0.25) (layer "B.Cu") (net 1))
   (segment (start 208.5 41.75) (end 209.123 41.127) (width 0.381) (layer "B.Cu") (net 1))
   (segment (start 210.813638 39.813362) (end 211.87825 39.813362) (width 0.381) (layer "B.Cu") (net 1))
@@
   (segment (start 208.601042 84.75) (end 207.7625 84.75) (width 0.3) (layer "B.Cu") (net 1))
   (segment (start 209.15 85.35) (end 209.15 85.298958) (width 0.3) (layer "B.Cu") (net 1))
+  (segment (start 199.4375 80.25) (end 201.35 80.25) (width 0.25) (layer "B.Cu") (net 1))
   (segment (start 208.45 77.05) (end 208.15 77.05) (width 0.6) (layer "B.Cu") (net 1))
   (segment (start 198.44 78.85) (end 198.1005 79.1895) (width 0.6) (layer "B.Cu") (net 1))
@@
   (segment (start 221.5 42.507) (end 222.13 42.507) (width 0.6) (layer "B.Cu") (net 1))
   (segment (start 198.1005 79.751542) (end 198.1005 79.723488) (width 0.3) (layer "B.Cu") (net 1))
+  (segment (start 202.85 83.25) (end 203.6 82.5) (width 0.25) (layer "B.Cu") (net 1))
+  (segment (start 202.85 86.6625) (end 202.85 83.25) (width 0.25) (layer "B.Cu") (net 1))
   (segment (start 222.12 39.597) (end 222.15 39.627) (width 0.6) (layer "B.Cu") (net 1))
   (segment (start 209.15 85.298958) (end 208.601042 84.75) (width 0.3) (layer "B.Cu") (net 1))
   (segment (start 222.13 42.507) (end 222.15 42.527) (width 0.6) (layer "B.Cu") (net 1))
+  (segment (start 207.7625 84.75) (end 205.85 84.75) (width 0.25) (layer "B.Cu") (net 1))
   (segment (start 209.15 85.35) (end 209.15 85.8) (width 0.6) (layer "B.Cu") (net 1))
   (segment (start 207.25 77.32) (end 207.25 77.15) (width 0.6) (layer "B.Cu") (net 1))
   (segment (start 207.25 88.06) (end 206.71 88.06) (width 0.6) (layer "B.Cu") (net 1))
   (segment (start 199.4375 80.25) (end 198.598958 80.25) (width 0.3) (layer "B.Cu") (net 1))
+  (segment (start 205.85 84.75) (end 203.6 82.5) (width 0.25) (layer "B.Cu") (net 1))
   (segment (start 203.6 81.426042) (end 203.6 82.5) (width 0.3) (layer "B.Cu") (net 1))
   (segment (start 221.5 39.597) (end 222.12 39.597) (width 0.6) (layer "B.Cu") (net 1))
@@
   (segment (start 208.12125 30.7975) (end 212.88375 59.3725) (width 0.6) (layer "F.Cu") (net 64))
   (segment (start 212.88375 59.3725) (end 215.265 87.9475) (width 0.6) (layer "F.Cu") (net 64))
+  (segment (start 211.5675 84.25) (end 207.7625 84.25) (width 0.25) (layer "B.Cu") (net 64))
+  (segment (start 215.265 87.9475) (end 211.5675 84.25) (width 0.25) (layer "B.Cu") (net 64))
   (segment (start 235.481726 86.780774) (end 234.315 87.9475) (width 0.6) (layer "F.Cu") (net 65))
+  (segment (start 234.315 80.3275) (end 233.3625 79.375) (width 0.25) (layer "F.Cu") (net 65))
   (segment (start 234.315 30.7975) (end 235.481726 31.964226) (width 0.6) (layer "F.Cu") (net 65))
   (segment (start 235.481726 31.964226) (end 235.481726 86.780774) (width 0.6) (layer "F.Cu") (net 65))
+  (segment (start 234.315 87.9475) (end 234.315 80.3275) (width 0.25) (layer "F.Cu") (net 65))
+  (via (at 233.3625 79.375) (size 0.8) (drill 0.4) (layers "F.Cu" "B.Cu") (net 65))
+  (segment (start 212.316116 82.75) (end 207.7625 82.75) (width 0.25) (layer "B.Cu") (net 65))
+  (segment (start 214.897366 80.16875) (end 212.316116 82.75) (width 0.25) (layer "B.Cu") (net 65))
+  (segment (start 232.56875 80.16875) (end 214.897366 80.16875) (width 0.25) (layer "B.Cu") (net 65))
+  (segment (start 233.3625 79.375) (end 232.56875 80.16875) (width 0.25) (layer "B.Cu") (net 65))
   (segment (start 253.365 30.7975) (end 254.531726 31.964226) (width 0.6) (layer "F.Cu") (net 66))
   (segment (start 254.531726 31.964226) (end 254.531726 86.780774) (width 0.6) (layer "F.Cu") (net 66))
   (segment (start 254.531726 86.780774) (end 253.365 87.9475) (width 0.6) (layer "F.Cu") (net 66))
+  (segment (start 247.1425 81.725) (end 236.16538 81.725) (width 0.25) (layer "B.Cu") (net 66))
+  (segment (start 213.1125 83.75) (end 207.7625 83.75) (width 0.25) (layer "B.Cu") (net 66))
+  (segment (start 236.16538 81.725) (end 235.91538 81.475) (width 0.25) (layer "B.Cu") (net 66))
+  (segment (start 253.365 87.9475) (end 247.1425 81.725) (width 0.25) (layer "B.Cu") (net 66))
+  (segment (start 235.91538 81.475) (end 215.3875 81.475) (width 0.25) (layer "B.Cu") (net 66))
+  (segment (start 215.3875 81.475) (end 213.1125 83.75) (width 0.25) (layer "B.Cu") (net 66))
   (segment (start 212.7 83.25) (end 207.7625 83.25) (width 0.3) (layer "B.Cu") (net 67))
   (segment (start 237.2 80.85) (end 243.4 80.85) (width 0.6) (layer "B.Cu") (net 67))
