File: cursed-scandinavian-iso-van.kicad_sch (KiCad schematic)
At the start: 102 parts, among them J1 Conn_01x04, SW1 SW_Push, U1 ATmega32U4-A, Y1 16MHz

Commit message: begun routing
Parts:
- added S1: MX_stab, PCM_marbastlib-mx:STAB_MX_P_3u, symbol PCM_marbastlib-mx:MX_stab
- added S2: MX_stab, PCM_marbastlib-mx:STAB_MX_P_2.75u, symbol PCM_marbastlib-mx:MX_stab
- added S3: MX_stab, PCM_marbastlib-mx:STAB_MX_P_ISO-ROT, symbol PCM_marbastlib-mx:MX_stab
- MX37, MX40: footprint PCM_marbastlib-mx:SW_MX_HS_1u -> PCM_marbastlib-mx:SW_MX_HS_1.25u
Changed lines of the file:
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@@
+    )
+  )
+  (symbol (lib_id "PCM_marbastlib-mx:MX_stab") (at 172.466 129.1336 0) (unit 1)
+    (in_bom yes) (on_board yes) (dnp no) (fields_autoplaced)
+    (property "Reference" "S2" (at 178.308 127.7366 0)
+      (effects (font (size 1.27 1.27)) (justify left))
+    )
+    (property "Value" "MX_stab" (at 178.308 130.2766 0)
+      (effects (font (size 1.27 1.27)) (justify left))
+    )
+    (property "Footprint" "PCM_marbastlib-mx:STAB_MX_P_2.75u" (at 172.466 129.1336 0)
+      (effects (font (size 1.27 1.27)) hide)
+    )
+    (property "Datasheet" "" (at 172.466 129.1336 0)
+      (effects (font (size 1.27 1.27)) hide)
+    )
+    (instances
+      (project "cursed-scandinavian-iso-van"
+        (path "/8f7563d1-5dae-4dee-af26-f72de8ce492b"
+          (reference "S2") (unit 1)
+        )
+      )
     )
   )
@@
       (effects (font (size 1.27 1.27)))
     )
-    (property "Footprint" "PCM_marbastlib-mx:SW_MX_HS_1u" (at 114.8588 101.9556 0)
+    (property "Footprint" "PCM_marbastlib-mx:SW_MX_HS_1.25u" (at 114.8588 101.9556 0)
       (effects (font (size 1.27 1.27)) hide)
     )
@@
         (path "/8f7563d1-5dae-4dee-af26-f72de8ce492b"
           (reference "D22") (unit 1)
+        )
+      )
+    )
+  )
+  (symbol (lib_id "PCM_marbastlib-mx:MX_stab") (at 197.2564 128.6764 0) (unit 1)
+    (in_bom yes) (on_board yes) (dnp no) (fields_autoplaced)
+    (property "Reference" "S3" (at 203.0984 127.2794 0)
+      (effects (font (size 1.27 1.27)) (justify left))
+    )
+    (property "Value" "MX_stab" (at 203.0984 129.8194 0)
+      (effects (font (size 1.27 1.27)) (justify left))
+    )
+    (property "Footprint" "PCM_marbastlib-mx:STAB_MX_P_ISO-ROT" (at 197.2564 128.6764 0)
+      (effects (font (size 1.27 1.27)) hide)
+    )
+    (property "Datasheet" "" (at 197.2564 128.6764 0)
+      (effects (font (size 1.27 1.27)) hide)
+    )
+    (instances
+      (project "cursed-scandinavian-iso-van"
+        (path "/8f7563d1-5dae-4dee-af26-f72de8ce492b"
+          (reference "S3") (unit 1)
         )
       )
@@
     )
   )
+  (symbol (lib_id "PCM_marbastlib-mx:MX_stab") (at 145.288 128.4732 0) (unit 1)
+    (in_bom yes) (on_board yes) (dnp no) (fields_autoplaced)
+    (property "Reference" "S1" (at 151.13 127.0762 0)
+      (effects (font (size 1.27 1.27)) (justify left))
+    )
+    (property "Value" "MX_stab" (at 151.13 129.6162 0)
+      (effects (font (size 1.27 1.27)) (justify left))
+    )
+    (property "Footprint" "PCM_marbastlib-mx:STAB_MX_P_3u" (at 145.288 128.4732 0)
+      (effects (font (size 1.27 1.27)) hide)
+    )
+    (property "Datasheet" "" (at 145.288 128.4732 0)
+      (effects (font (size 1.27 1.27)) hide)
+    )
+    (instances
+      (project "cursed-scandinavian-iso-van"
+        (path "/8f7563d1-5dae-4dee-af26-f72de8ce492b"
+          (reference "S1") (unit 1)
+        )
+      )
+    )
+  )
   (symbol (lib_id "Device:D_Small") (at 193.5988 66.3956 90) (unit 1)
     (in_bom yes) (on_board yes) (dnp no) (fields_autoplaced)
@@
       (effects (font (size 1.27 1.27)))
     )
-    (property "Footprint" "PCM_marbastlib-mx:SW_MX_HS_1u" (at 221.5388 101.9556 0)
-      (effects (font (size 1.27 1.27)) hide)
-    )
+    (property "Footprint" "PCM_marbastlib-mx:SW_MX_HS_1.25u" (at 221.5388 101.9556 0)
+      (effects (font (size 1.27 1.27)) hide)
+    )

Commit message: maybe all the columns
Connections:
- net COL0: now also U1.8 (PB0)
- net COL1: now also U1.9 (PB1)
- net COL10: now also U1.30 (PB6)
- net COL11: now also U1.31 (PC6)
- net COL2: now also U1.10 (PB2)
- net COL3: now also U1.11 (PB3)
- net COL4: now also U1.18 (PD0)
- net COL5: now also U1.19 (PD1)
- net COL6: now also U1.20 (PD2)
- net COL7: now also U1.21 (PD3)
- net COL8: now also U1.22 (PD5)
- net COL9: now also U1.29 (PB5)
- net GND: now also SW1.2; no longer SW1.1
- net ROW3: now also U1.32 (PC7)
- net at R1.2, U1.13 (~{RESET}): now also SW1.1; no longer SW1.2
Changed lines of the file:
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@@
+    )
+  )
+  (global_label "COL9" (shape input) (at 61.4172 45.3136 0) (fields_autoplaced)
+    (effects (font (size 1.27 1.27)) (justify left))
+    (property "Intersheetrefs" "${INTERSHEET_REFS}" (at 69.2405 45.3136 0)
+      (effects (font (size 1.27 1.27)) (justify left) hide)
     )
   )
@@
     )
   )
+  (global_label "COL8" (shape input) (at 61.4172 75.7936 0) (fields_autoplaced)
+    (effects (font (size 1.27 1.27)) (justify left))
+    (property "Intersheetrefs" "${INTERSHEET_REFS}" (at 69.2405 75.7936 0)
+      (effects (font (size 1.27 1.27)) (justify left) hide)
+    )
+  )
   (global_label "COL9" (shape input) (at 234.2896 28.2448 90) (fields_autoplaced)
     (effects (font (size 1.27 1.27)) (justify left))
@@
     )
   )
+  (global_label "COL10" (shape input) (at 61.4172 47.8536 0) (fields_autoplaced)
+    (effects (font (size 1.27 1.27)) (justify left))
+    (property "Intersheetrefs" "${INTERSHEET_REFS}" (at 70.45 47.8536 0)
+      (effects (font (size 1.27 1.27)) (justify left) hide)
+    )
+  )
+  (global_label "COL0" (shape input) (at 61.4172 32.6136 0) (fields_autoplaced)
+    (effects (font (size 1.27 1.27)) (justify left))
+    (property "Intersheetrefs" "${INTERSHEET_REFS}" (at 69.2405 32.6136 0)
+      (effects (font (size 1.27 1.27)) (justify left) hide)
+    )
+  )
+  (global_label "COL3" (shape input) (at 61.4172 40.2336 0) (fields_autoplaced)
+    (effects (font (size 1.27 1.27)) (justify left))
+    (property "Intersheetrefs" "${INTERSHEET_REFS}" (at 69.2405 40.2336 0)
+      (effects (font (size 1.27 1.27)) (justify left) hide)
+    )
+  )
   (global_label "COL5" (shape input) (at 173.3296 28.2448 90) (fields_autoplaced)
     (effects (font (size 1.27 1.27)) (justify left))
     (property "Intersheetrefs" "${INTERSHEET_REFS}" (at 173.3296 20.4215 90)
+      (effects (font (size 1.27 1.27)) (justify left) hide)
+    )
+  )
+  (global_label "COL11" (shape input) (at 61.4172 55.4736 0) (fields_autoplaced)
+    (effects (font (size 1.27 1.27)) (justify left))
+    (property "Intersheetrefs" "${INTERSHEET_REFS}" (at 70.45 55.4736 0)
       (effects (font (size 1.27 1.27)) (justify left) hide)
     )
@@
     )
   )
+  (global_label "COL6" (shape input) (at 61.4172 68.1736 0) (fields_autoplaced)
+    (effects (font (size 1.27 1.27)) (justify left))
+    (property "Intersheetrefs" "${INTERSHEET_REFS}" (at 69.2405 68.1736 0)
+      (effects (font (size 1.27 1.27)) (justify left) hide)
+    )
+  )
   (global_label "XTAL2" (shape input) (at 30.9372 42.7736 180) (fields_autoplaced)
     (effects (font (size 1.27 1.27)) (justify right))
@@
     )
   )
+  (global_label "COL4" (shape input) (at 61.4172 63.0936 0) (fields_autoplaced)
+    (effects (font (size 1.27 1.27)) (justify left))
+    (property "Intersheetrefs" "${INTERSHEET_REFS}" (at 69.2405 63.0936 0)
+      (effects (font (size 1.27 1.27)) (justify left) hide)
+    )
+  )
+  (global_label "COL2" (shape input) (at 61.4172 37.6936 0) (fields_autoplaced)
+    (effects (font (size 1.27 1.27)) (justify left))
+    (property "Intersheetrefs" "${INTERSHEET_REFS}" (at 69.2405 37.6936 0)
+      (effects (font (size 1.27 1.27)) (justify left) hide)
+    )
+  )
   (global_label "COL1" (shape input) (at 112.3696 28.2448 90) (fields_autoplaced)
     (effects (font (size 1.27 1.27)) (justify left))
     (property "Intersheetrefs" "${INTERSHEET_REFS}" (at 112.3696 20.4215 90)
+      (effects (font (size 1.27 1.27)) (justify left) hide)
+    )
+  )
+  (global_label "COL5" (shape input) (at 61.4172 65.6336 0) (fields_autoplaced)
+    (effects (font (size 1.27 1.27)) (justify left))
+    (property "Intersheetrefs" "${INTERSHEET_REFS}" (at 69.2405 65.6336 0)
       (effects (font (size 1.27 1.27)) (justify left) hide)
     )
@@
     (property "Intersheetrefs" "${INTERSHEET_REFS}" (at 83.7522 48.6156 0)
       (effects (font (size 1.27 1.27)) (justify right) hide)
+    )
+  )
+  (global_label "ROW3" (shape input) (at 61.4172 58.0136 0) (fields_autoplaced)
+    (effects (font (size 1.27 1.27)) (justify left))
+    (property "Intersheetrefs" "${INTERSHEET_REFS}" (at 69.6638 58.0136 0)
+      (effects (font (size 1.27 1.27)) (justify left) hide)
+    )
+  )
+  (global_label "COL7" (shape input) (at 61.4172 70.7136 0) (fields_autoplaced)
+    (effects (font (size 1.27 1.27)) (justify left))
+    (property "Intersheetrefs" "${INTERSHEET_REFS}" (at 69.2405 70.7136 0)
+      (effects (font (size 1.27 1.27)) (justify left) hide)
+    )
+  )
+  (global_label "COL1" (shape input) (at 61.4172 35.1536 0) (fields_autoplaced)
+    (effects (font (size 1.27 1.27)) (justify left))
+    (property "Intersheetrefs" "${INTERSHEET_REFS}" (at 69.2405 35.1536 0)
+      (effects (font (size 1.27 1.27)) (justify left) hide)
     )
   )
@@
     )
   )
-  (symbol (lib_id "Switch:SW_Push") (at 23.7236 32.6136 0) (unit 1)
-    (in_bom yes) (on_board yes) (dnp no) (fields_autoplaced)
+  (symbol (lib_id "Switch:SW_Push") (at 23.7236 32.6136 0) (mirror y) (unit 1)
+    (in_bom yes) (on_board yes) (dnp no)
     (property "Reference" "SW1" (at 23.7236 24.9936 0)
       (effects (font (size 1.27 1.27)))

Commit message: only silk and edge complaints
Connections:
- net ROW0: now also U1.26 (PD6)
- net ROW1: now also U1.27 (PD7)
- net ROW2: now also U1.28 (PB4)
- no-connect marks 0 -> 10
Changed lines of the file:
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@@
   (junction (at 208.8388 68.9356) (diameter 0) (color 0 0 0 0)
   )
+  (no_connect (at 61.4172 50.3936))
+  (no_connect (at 61.4172 93.5736))
+  (no_connect (at 61.4172 98.6536))
+  (no_connect (at 61.4172 73.2536))
+  (no_connect (at 61.4172 103.7336))
+  (no_connect (at 61.4172 106.2736))
+  (no_connect (at 61.4172 96.1136))
+  (no_connect (at 61.4172 88.4936))
+  (no_connect (at 61.4172 101.1936))
+  (no_connect (at 30.9372 47.8536))
   (wire (pts (xy 188.5696 28.9052) (xy 188.5188 28.9052))
     (stroke (width 0) (type default))
@@
     )
   )
+  (global_label "ROW1" (shape input) (at 61.4172 80.8736 0) (fields_autoplaced)
+    (effects (font (size 1.27 1.27)) (justify left))
+    (property "Intersheetrefs" "${INTERSHEET_REFS}" (at 69.6638 80.8736 0)
+      (effects (font (size 1.27 1.27)) (justify left) hide)
+    )
+  )
   (global_label "D+" (shape input) (at 22.7076 178.4096 180) (fields_autoplaced)
     (effects (font (size 1.27 1.27)) (justify right))
@@
     )
   )
+  (global_label "ROW2" (shape input) (at 61.4172 42.7736 0) (fields_autoplaced)
+    (effects (font (size 1.27 1.27)) (justify left))
+    (property "Intersheetrefs" "${INTERSHEET_REFS}" (at 69.6638 42.7736 0)
+      (effects (font (size 1.27 1.27)) (justify left) hide)
+    )
+  )
   (global_label "COL10" (shape input) (at 61.4172 47.8536 0) (fields_autoplaced)
     (effects (font (size 1.27 1.27)) (justify left))
@@
     )
   )
+  (global_label "ROW0" (shape input) (at 61.4172 78.3336 0) (fields_autoplaced)
+    (effects (font (size 1.27 1.27)) (justify left))
+    (property "Intersheetrefs" "${INTERSHEET_REFS}" (at 69.6638 78.3336 0)
+      (effects (font (size 1.27 1.27)) (justify left) hide)
+    )
+  )

Commit message: second attempt
Parts:
- removed U1: ATmega32U4-A, Package_QFP:TQFP-44_10x10mm_P0.8mm, symbol MCU_Microchip_ATmega:ATmega32U4-A
- added U1: ATmega32U4-M, Package_DFN_QFN:QFN-44-1EP_7x7mm_P0.5mm_EP5.2x5.2mm, symbol MCU_Microchip_ATmega:ATmega32U4-M
- C1, C2, C3, C4, C5, C6, C7: footprint Capacitor_SMD:C_0805_2012Metric -> Capacitor_SMD:C_0402_1005Metric
- R1, R2, R3, R4: footprint Resistor_SMD:R_0805_2012Metric -> Resistor_SMD:R_0402_1005Metric
Connections:
- net +5V: now also U1.14 (VCC), U1.2 (UVCC), U1.24 (AVCC), U1.34 (VCC), U1.44 (AVCC), U1.7 (VBUS)
- net COL0: now also U1.25 (PD4)
- net COL1: now also U1.26 (PD6)
- net COL10: now also U1.19 (PD1)
- net COL11: now also U1.20 (PD2)
- net COL2: now also U1.27 (PD7)
- net COL3: now also U1.28 (PB4)
- net COL4: now also U1.29 (PB5)
- net COL5: now also U1.30 (PB6)
- net COL6: now also U1.31 (PC6)
- net COL7: now also U1.32 (PC7)
- net COL8: now also U1.21 (PD3)
- net COL9: now also U1.18 (PD0)
- net GND: now also U1.15 (GND), U1.23 (GND), U1.35 (GND), U1.43 (GND), U1.45 (GND), U1.5 (UGND)
- net ROW0: now also U1.38 (PF5)
- net ROW1: now also U1.37 (PF6)
- net ROW2: now also U1.36 (PF7)
- net ROW3: now also U1.22 (PD5)
- net XTAL1: now also U1.17 (XTAL1)
- net XTAL2: now also U1.16 (XTAL2)
- net at R1.2, SW1.1: now also U1.13 (~{RESET})
- net at R3.2: now also U1.3 (D-)
- net at R4.1: now also U1.33 (~{HWB}/PE2)
- net at R2.2: now also U1.4 (D+)
- net at C1.1: now also U1.6 (UCAP)
- no-connect marks 10 -> 1

Commit message: maybe
Parts:
- removed F1: 500mA, Fuse:Fuse_1206_3216Metric, symbol Device:Polyfuse_Small
- removed R2, R3: 22, Resistor_SMD:R_0402_1005Metric, symbol Device:R_Small
- removed R4: 10k, Resistor_SMD:R_0402_1005Metric, symbol Device:R_Small
- removed U1: ATmega32U4-M, Package_DFN_QFN:QFN-44-1EP_7x7mm_P0.5mm_EP5.2x5.2mm, symbol MCU_Microchip_ATmega:ATmega32U4-M
- removed Y1: 16MHz, Crystal:Crystal_SMD_3225-4Pin_3.2x2.5mm, symbol Device:Crystal_GND24_Small
- added C8, C9: 1uF, Capacitor_SMD:C_0402_1005Metric, symbol Device:C_Small
- added U1: STM32F072CBTx, Package_QFP:LQFP-48_7x7mm_P0.5mm, symbol MCU_ST_STM32F0:STM32F072CBTx
- added U2: XC6206PxxxMR, Package_TO_SOT_SMD:SOT-23-3, symbol Regulator_Linear:XC6206PxxxMR
- C1: value 1u -> 100nF
- C2, C3: value 22p -> 100nF
- C4, C5, C6: value 0.1u -> 100nF
- C7: value 10u -> 10uF; footprint Capacitor_SMD:C_0402_1005Metric -> Capacitor_SMD:C_0603_1608Metric
- SW1: footprint Button_Switch_SMD:SW_SPST_TL3342 -> Button_Switch_SMD:SW_SPST_SKQG_WithoutStem
Connections:
- net VCC is gone; now on net +5V: J1.1 (Pin_1)
- net XTAL1 is gone; now on net GND: C2.2
- net XTAL2 is gone; now on net GND: C3.2
- net +5V: now also C8.1, U2.3 (VI); no longer C4.1, C5.1, C6.1, C7.1, R1.1
- net COL0: now also U1.13 (PA3)
- net COL1: now also U1.14 (PA4)
- net COL10: now also U1.4 (PC15)
- net COL11: now also U1.3 (PC14)
- net COL2: now also U1.15 (PA5)
- net COL3: now also U1.16 (PA6)
- net COL4: now also U1.17 (PA7)
- net COL5: now also U1.18 (PB0)
- net COL6: now also U1.19 (PB1)
- net COL7: now also U1.20 (PB2)
- net COL8: now also U1.21 (PB10)
- net COL9: now also U1.25 (PB12)
- net GND: now also R1.2, C8.2, C9.2, U1.23 (VSS), U1.35 (VSS), U1.47 (VSS), U1.8 (VSSA), U2.1 (GND); no longer C2.1, C3.1, SW1.2
- net ROW0: now also U1.26 (PB13)
- net ROW1: now also U1.12 (PA2)
- net ROW2: now also U1.11 (PA1)
- net ROW3: now also U1.10 (PA0)
- net +3.3V: now reaches SW1.1
- net +3.3V: now also C2.1, C3.1, C4.1, C5.1, C6.1, C7.1, C9.1, U1.1 (VBAT), U1.24 (VDD), U1.36 (VDDIO2), U1.48 (VDD), U1.9 (VDDA), U2.2 (VO); no longer R1.2
- net NRST: now reaches C1.1
- net NRST: now also U1.7 (NRST)
- net D+ renamed D_P
- net D_P: now also U1.33 (PA12)
- net D- renamed D_N
- net D_N: now also U1.32 (PA11)
- new net BOOT0: R1.1, SW1.2, U1.44 (BOOT0)
- no-connect marks 1 -> 0
Other:
- moved on the sheet: C4, C5, C6, C7
