File: cursed-scandinavian-iso-van.kicad_sch (KiCad schematic)
At the start: 105 parts, among them J1 Conn_01x04, SW1 SW_Push, U1 ATmega32U4-M, Y1 16MHz

Commit message: finish PCB in STM32
Parts:
- removed C1: 1u, Capacitor_SMD:C_0402_1005Metric, symbol Device:C_Small
- removed C2, C3: 22p, Capacitor_SMD:C_0402_1005Metric, symbol Device:C_Small
- removed C4, C5, C6: 0.1u, Capacitor_SMD:C_0402_1005Metric, symbol Device:C_Small
- removed C7: 10u, Capacitor_SMD:C_0402_1005Metric, symbol Device:C_Small
- removed F1: 500mA, Fuse:Fuse_1206_3216Metric, symbol Device:Polyfuse_Small
- removed J1: Conn_01x04, Connector_JST:JST_SH_SM04B-SRSS-TB_1x04-1MP_P1.00mm_Horizontal, symbol Connector_Generic:Conn_01x04
- removed R1, R4: 10k, Resistor_SMD:R_0402_1005Metric, symbol Device:R_Small
- removed R2, R3: 22, Resistor_SMD:R_0402_1005Metric, symbol Device:R_Small
- removed SW1: SW_Push, Button_Switch_SMD:SW_SPST_TL3342, symbol Switch:SW_Push
- removed U1: ATmega32U4-M, Package_DFN_QFN:QFN-44-1EP_7x7mm_P0.5mm_EP5.2x5.2mm, symbol MCU_Microchip_ATmega:ATmega32U4-M
- removed Y1: 16MHz, Crystal:Crystal_SMD_3225-4Pin_3.2x2.5mm, symbol Device:Crystal_GND24_Small
- added C? (x2): 1uF, Capacitor_SMD:C_0402_1005Metric, symbol Device:C_Small
- added C? (x6): 100nF, Capacitor_SMD:C_0402_1005Metric, symbol Device:C
- added C?: 10uF, Capacitor_SMD:C_0603_1608Metric, symbol Device:C
- added C?: 100nF, Capacitor_SMD:C_0402_1005Metric, symbol Device:C_Small
- added F1: ASMD1206-150, Fuse:Fuse_1206_3216Metric, symbol Device:Polyfuse
- added J2: Conn_01x04_Socket, Connector_JST:JST_SH_SM04B-SRSS-TB_1x04-1MP_P1.00mm_Horizontal, symbol Connector:Conn_01x04_Socket
- added R?: 10k, Resistor_SMD:R_0402_1005Metric, symbol Device:R_Small
- added SW?: SKQGABE010, Button_Switch_SMD:SW_SPST_SKQG_WithoutStem, symbol Switch:SW_Push
- added U1: STM32F072CBU6, Package_QFP:LQFP-48-1EP_7x7mm_P0.5mm_EP3.6x3.6mm, symbol MCU_ST_STM32F0:STM32F072CBUx
- added U2: PRTR5V0U2X, Package_TO_SOT_SMD:SOT-143, symbol Power_Protection:PRTR5V0U2X
- added U?: XC6206P332MR-Regulator_Linear, Package_TO_SOT_SMD:SOT-23, symbol kicad-keyboard-parts:XC6206PxxxMR-Regulator_Linear
Connections:
- net +5V: now also C?.1, C?.2, F1.2, U2.4 (VCC), U?.3 (VI)
- net GND: now also C?.1, C?.1, C?.2, C?.2, C?.2, C?.2, C?.2, C?.2, C?.2, C?.2, J2.4 (Pin_4), R?.2, U1.23 (VSS), U1.35 (VSS), U1.47 (VSS), U1.49 (VSS), U1.8 (VSSA), U2.1 (GND), U?.1 (GND)
- net COL0 renamed col0
- net col0: now also U1.22 (PB11)
- net COL1 renamed col1
- net col1: now also U1.21 (PB10)
- net COL10 renamed col10
- net COL11 renamed col11
- net COL2 renamed col2
- net col2: now also U1.20 (PB2)
- net COL3 renamed col3
- net col3: now also U1.19 (PB1)
- net COL4 renamed col4
- net col4: now also U1.18 (PB0)
- net COL5 renamed col5
- net col5: now also U1.17 (PA7)
- net COL6 renamed col6
- net col6: now also U1.16 (PA6)
- net COL7 renamed col7
- net col7: now also U1.15 (PA5)
- net COL8 renamed col8
- net col8: now also U1.14 (PA4)
- net COL9 renamed col9
- net ROW0 renamed row0
- net row0: now also U1.26 (PB13)
- net ROW1 renamed row1
- net row1: now also U1.34 (PA13)
- net ROW2 renamed row2
- net row2: now also U1.25 (PB12)
- net ROW3 renamed row3
- net row3: now also U1.13 (PA3)
- new net +3V3: C?.1, C?.1, C?.1, C?.1, C?.1, C?.1, C?.2, SW?.1, U1.1 (VBAT), U1.24 (VDD), U1.36 (VDDIO2), U1.48 (VDD), U1.9 (VDDA), U?.2 (VO)
- new net A0: U1.10 (PA0)
- new net A1: U1.11 (PA1)
- new net A10: U1.31 (PA10)
- new net A14: U1.37 (PA14)
- new net A15: U1.38 (PA15)
- new net A2: U1.12 (PA2)
- new net A8: U1.29 (PA8)
- new net A9: U1.30 (PA9)
- new net B14: U1.27 (PB14)
- new net B15: U1.28 (PB15)
- new net B3: U1.39 (PB3)
- new net B4: U1.40 (PB4)
- new net B5: U1.41 (PB5)
- new net B6: U1.42 (PB6)
- new net B7: U1.43 (PB7)
- new net B8: U1.45 (PB8)
- new net B9: U1.46 (PB9)
- new net BOOT0: R?.1, SW?.2, U1.44 (BOOT0)
- new net D_N: J2.2 (Pin_2), U1.32 (PA11), U2.2 (I/O1)
- new net D_P: J2.3 (Pin_3), U1.33 (PA12), U2.3 (I/O2)
- new net NRST: C?.1, U1.7 (NRST)
- new net VBUS: F1.1, J2.1 (Pin_1)
- no-connect marks 1 -> 5
Other:
- note added: "3.3V LDO"
- note added: "Differntial pair ref: 2 layer PCB microstrip spacing: 0.127mm coplanar reference spacing: 0.127mm signal width: 0.25mm dielectric thickness: 1.6mm calculator: https://www.eeweb.com/tools/edge-coupled-microstrip-impedance/ https://resources.altium.com/p/routing-requirements-usb-20-2-layer-pcb"
- note added: "Key Matrix"
- note added: "MCU"
- note added: "Matrix Pinout"
- note added: "NRST has internal pull up Hold high for normal operation"
- note added: "OLED display"
- note added: "RGB LEDs"
- note added: "Trackpoint"
- note added: "USB-C and ESD"
- note added: "button to pull boot0 high while reseting to activate DFU"
- moved on the sheet: D1, D10, D11, D12, D13, D14, D15, D16, D17, D18, D19, D2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

Commit message: updated PCB
Connections:
- net B7 is gone; now on net col10: U1.43 (PB7)
- net B8 is gone; now on net col11: U1.45 (PB8)
- net B9 is gone; now on net col9: U1.46 (PB9)
Changed lines of the file:
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@@
     (stroke (width 0) (type default))
   )
-  (wire (pts (xy 156.21 53.34) (xy 159.131 53.34))
+  (wire (pts (xy 156.21 53.34) (xy 159.385 53.34))
     (stroke (width 0) (type default))
   )
@@
     (effects (font (size 1.27 1.27)) (justify right bottom))
   )
+  (label "B7" (at 159.385 53.34 0) (fields_autoplaced)
+    (effects (font (size 1.27 1.27)) (justify left bottom))
+  )
   (label "A14" (at 61.976 73.914 0) (fields_autoplaced)
     (effects (font (size 1.27 1.27)) (justify left bottom))
@@
     (effects (font (size 1.27 1.27)) (justify left bottom))
   )
-  (label "A" (at 159.385 50.8 0) (fields_autoplaced)
-    (effects (font (size 1.27 1.27)) (justify left bottom))
-  )
+  (label "B9" (at 159.385 50.8 0) (fields_autoplaced)
+    (effects (font (size 1.27 1.27)) (justify left bottom))
+  )
+  (label "B8" (at 159.385 55.88 0) (fields_autoplaced)
+    (effects (font (size 1.27 1.27)) (justify left bottom))
+  )
